File: ATTiny85 Light 2.kicad_pcb (KiCad board)
At the start: 2 copper layers, 40 x 45 mm, 4 parts

Commit message: Add files via upload
Routing:
- net Net-(R2-Pad1): track 45.7 -> 47.1 mm
Other:
- board text added: "LED V1.1"
- board text removed: "LED V1.0"

Commit message: Add files via upload
Parts:
- added H1: MountingHole, MountingHole:MountingHole_2.2mm_M2, F.Cu at (114.2, 76.2)
- added H2: MountingHole_Pad, MountingHole:MountingHole_2.2mm_M2_DIN965_Pad, F.Cu at (97.8, 91.3)
- added H3: MountingHole_Pad, MountingHole:MountingHole_2.2mm_M2_DIN965_Pad, F.Cu at (130.3, 86.4)
- added H4: MountingHole, MountingHole:MountingHole_2.2mm_M2, F.Cu at (130.4, 114.3)
- added H5: MountingHole_Pad, MountingHole:MountingHole_2.2mm_M2_DIN965_Pad, F.Cu at (102.0, 85.1)
- added H6: MountingHole, MountingHole:MountingHole_2.2mm_M2, F.Cu at (97.3, 114.2)
- added H7: MountingHole_Pad, MountingHole:MountingHole_2.2mm_M2_DIN965_Pad, F.Cu at (126.3, 81.0)
- R1: renamed from R 220
- R3: renamed from R 10k
- renumbered LDR to R2, ATTiny85 to U1
Connections:
- net VDC renamed VCC
Routing:
- net Net-(R2-Pad1): track 47.1 -> 48.5 mm
- net VCC: track 22.6 -> 22.9 mm, vias 1 -> 0
- net Net-(H5-Pad1): vias 1 -> 0
- net GND: vias 2 -> 0
- net (no net): vias 3 -> 0
Other:
- board text removed: "+"
- board text removed: "-"
- board text removed: "GND"
- board text removed: "VCC"

Commit message: Add files via upload
Parts:
- removed H2, H3, H5, H7: MountingHole_Pad, MountingHole:MountingHole_2.2mm_M2_DIN965_Pad
- added BATT+: MountingHole_Pad, MountingHole:MountingHole_2.2mm_M2_DIN965_Pad, F.Cu at (126.0, 81.0)
- added BATT-: MountingHole_Pad, MountingHole:MountingHole_2.2mm_M2_DIN965_Pad, F.Cu at (129.9, 86.4)
- added LED+: MountingHole_Pad, MountingHole:MountingHole_2.2mm_M2_DIN965_Pad, F.Cu at (102.0, 86.0)
- added LED-: MountingHole_Pad, MountingHole:MountingHole_2.2mm_M2_DIN965_Pad, F.Cu at (97.4, 92.5)
- LDR: renamed from R2; value R_PHOTO -> LDR
- R10k: renamed from R3; value R_Small -> R 220
- R220: renamed from R1; value R_Small -> R 10k
- renumbered U1 to ATTiny85
Other:
- board text removed: "Battery"
- board text removed: "LED"
